File: hardware/fluidnc-bob/fluidnc-bob.kicad_sch (KiCad schematic)
At the start: 45 parts, among them J1 5V-IN, J10 LIM-Z, J11 PROBE, J2 X-DRV, J3 Y-DRV, J4 Z-DRV, J5 LIM-X, J6 LIM-Y, J7 RELAY, J8 AUX, J9 SD, Q1 MMBT2222A, U1 SN74HC541N

Commit message: Layout updated
Parts:
- removed J9: SD, fluidnc-bob:WirePads_1x06_P5.08mm, symbol bob:PadS_06
- added J13: Conn_02x06_Odd_Even, Connector_PinHeader_2.54mm:PinHeader_2x06_P2.54mm_Vertical, symbol Connector_Generic:Conn_02x06_Odd_Even
Connections:
- net +5V: now also J13.5 (Pin_5)
- net GND: now also J13.11 (Pin_11), J13.12 (Pin_12)
- net at R32.2: now also A1.26 (GPIO1); no longer A1.28 (GPIO42)
- net at R30.2: now also A1.28 (GPIO42); no longer A1.26 (GPIO1)
- net CS: now reaches A1.16 (GPIO10)
- net CS: now also J13.10 (Pin_10)
- net MOSI: now reaches A1.17 (GPIO11)
- net MOSI: now also J13.8 (Pin_8)
- net SCK: now reaches A1.18 (GPIO12)
- net SCK: now also J13.9 (Pin_9)
- net MISO: now reaches A1.19 (GPIO13)
- net MISO: now also J13.7 (Pin_7)
- no-connect marks 22 -> 27
Other:
- moved on the sheet: A1, C2, C20, C22, D3, J10, J5, R20, R22, R30, R32

Commit message: Layout changed to shrink
Parts:
- added H1, H2, H3, H4: MountingHole, MountingHole:MountingHole_3.2mm_M3, symbol Mechanical:MountingHole
Connections:
- net GND: now also J1.1; no longer J1.2
- net at R14.1, U1.6 (A5): now also A1.7 (GPIO7); no longer A1.8 (GPIO15)
- net at F1.1: now also J1.2; no longer J1.1
- net at R16.1, U1.8 (A7): now also A1.5 (GPIO5); no longer A1.10 (GPIO17)
- net at R17.1, U1.9 (A8): now also A1.4 (GPIO4); no longer A1.11 (GPIO18)
- net at R10.1, U1.2 (A1): now also A1.11 (GPIO18); no longer A1.4 (GPIO4)
- net at R11.1, U1.3 (A2): now also A1.10 (GPIO17); no longer A1.5 (GPIO5)
- net at R12.1, U1.4 (A3): now also A1.9 (GPIO16); no longer A1.6 (GPIO6)
- net at R13.1, U1.5 (A4): now also A1.8 (GPIO15); no longer A1.7 (GPIO7)
- net at R15.1, U1.7 (A6): now also A1.6 (GPIO6); no longer A1.9 (GPIO16)
Other:
- moved on the sheet: C2, D3, U1
