File: hardware/fluidnc-bob-revD/fluidnc-bob-revD.kicad_sch (KiCad schematic)
At the start: 66 parts, among them J1 5V-IN, J10 SPINDLE-SW, J11 AUX, J13 SD, J2 EN+X, J3 X+Y, J4 Z+5, J5 LIM-X, J6 LIM-Y, J7 LIM-Z, J8 PROBE, J9 E-STOP, Q1 MMBT2222A, Q2 MMBT2222A, U1 SN74AHCT541N

Commit message: revD: board bring-up — as-built FluidNC config, R40 100R fix
- config.yaml for the as-built rev D pin map (verified against schematic
  netlist AND fabbed PCB pad nets): X step/dir gpio.7/6, Z gpio.18/17 —
  swapped vs rev C — spindle relay gpio.4, AUX gpio.5, estop gpio.8,
  shared EN gpio.9. estop_pin section commented until J9 is wired (NC
  input reads triggered when open -> critical alarm at boot).
- schematic: R40 (ZDIR series) 1k -> 100R to match its R60-R66 siblings;
  1k starves the FMD2740C opto input (~3 mA). Built board still has 1k —
  rework pending.
- Board flashed with FluidNC v4.0.4 wifi_s3, config loads clean, WebUI
  restored (release install-fs_s3.sh flashes littlefs to the wrong S3
  offset), hostname sharkcnc.local.

Co-Authored-By: Claude Fable 5 <noreply@anthropic.com>
Parts:
- R40: value 1k -> 100R
Changed lines of the file:
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@@
 	(wire
 		(pts
-			(xy 220.98 146.05) (xy 208.28 146.05)
-		)
-		(stroke
-			(width 0)
-			(type default)
-		)
-	)
-	(wire
-		(pts
 			(xy 158.75 133.35) (xy 160.02 133.35)
 		)
@@
 			)
 		)
-		(property "Value" "1k"
+		(property "Value" "100R"
 			(at 153.67 138.43 0)
 			(hide yes)
